File: _assembly/GL516_Template.kicad_pcb (KiCad board)
At the start: 2 copper layers, 304.8 x 99.2 mm, 98 parts, among them J1 Conn_01x02, J18 Conn_01x07, SW1 SW_PUSH, SW10 SW_PUSH, SW11 SW_PUSH, SW12 SW_PUSH, SW13 SW_PUSH, SW14 SW_PUSH, SW15 SW_PUSH, SW16 SW_PUSH, SW17 SW_PUSH, SW18 SW_PUSH, SW19 SW_PUSH, SW2 SW_PUSH, SW20 SW_PUSH, SW21 SW_PUSH, SW22 SW_PUSH, SW23 SW_PUSH, SW24 SW_PUSH, SW25 SW_PUSH, SW26 SW_PUSH, SW27 SW_PUSH, SW28 SW_PUSH, SW29 SW_PUSH, SW3 SW_PUSH, SW30 SW_PUSH, SW31 SW_PUSH, SW32 SW_PUSH, SW33 SW_PUSH, SW34 SW_PUSH, SW35 SW_PUSH, SW36 SW_PUSH, SW37 SW_PUSH, SW38 SW_PUSH, SW39 SW_PUSH, SW4 SW_PUSH, SW40 SW_PUSH, SW41 SW_PUSH, SW42 SW_PUSH, SW43 SW_PUSH, SW44 SW_PUSH, SW45 SW_PUSH, SW5 SW_PUSH, SW6 SW_PUSH, SW7 SW_PUSH, SW8 SW_PUSH, SW81 SW_PUSH, SW9 SW_PUSH, U1 BLEMicroPro

Commit message: PCB作成
Routing:
- net MOSI: track 0.00 -> 215.2 mm, vias 0 -> 5
- net Col6: track 40.1 -> 230.3 mm, vias 0 -> 4
- net MISO: track 0.00 -> 177.5 mm, vias 0 -> 1
- net Col0: track 217.2 -> 361.1 mm, vias 2 -> 3
- net MOTION: track 0.00 -> 135.3 mm, vias 0 -> 4
- net Row1: track 210.1 -> 336.5 mm, vias 0 -> 7
- net Col1: track 293.2 -> 417.8 mm, vias 2 -> 3
- net Row2: track 237.3 -> 355.2 mm, vias 0 -> 7
- net Col2: track 310.3 -> 415.8 mm, vias 4 -> 5
- net Row0: track 234.3 -> 336.5 mm, vias 0 -> 6
- net Row3: track 210.3 -> 308.2 mm
- net Col3: track 298.2 -> 376.5 mm, vias 4 -> 5
- net Col4: track 273.9 -> 333.6 mm, vias 4 -> 5
- net GND: track 0.00 -> 43.9 mm, vias 0 -> 2
- net Col5: track 284.0 -> 317.8 mm
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- added copper zone on B.Cu, net GND
- added copper zone on F.Cu, net GND

Commit message: トッププレート調整中
Changed lines of the file:
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@@
   )
   (setup
-    (last_trace_width 0.5)
+    (last_trace_width 0.25)
     (user_trace_width 0.5)
     (user_trace_width 0.5)
@@
     (visible_elements 7FFFFFFF)
     (pcbplotparams
-      (layerselection 0x01000_7ffffffe)
+      (layerselection 0x010fc_ffffffff)
       (usegerberextensions true)
       (usegerberattributes false)
@@
       (psa4output false)
       (plotreference true)
-      (plotvalue true)
+      (plotvalue false)
       (plotinvisibletext false)
       (padsonsilk false)
-      (subtractmaskfromsilk false)
-      (outputformat 3)
+      (subtractmaskfromsilk true)
+      (outputformat 1)
       (mirror false)
       (drillshape 0)
       (scaleselection 1)
-      (outputdirectory "./"))
+      (outputdirectory "./garber"))
   )
   (net 0 "")
@@
     (tags "mounting hole 2.2mm no annular m2")
     (attr virtual)
-    (fp_text reference REF** (at 0 -3.2) (layer F.SilkS)
+    (fp_text reference REF** (at 0 -3.2) (layer F.SilkS) hide
       (effects (font (size 1 1) (thickness 0.15)))
     )
@@
     (tags "mounting hole 2.2mm no annular m2")
     (attr virtual)
-    (fp_text reference REF** (at 0 -3.2) (layer F.SilkS)
+    (fp_text reference REF** (at 0 -3.2) (layer F.SilkS) hide
       (effects (font (size 1 1) (thickness 0.15)))
     )
@@
     (tags "mounting hole 2.2mm no annular m2")
     (attr virtual)
-    (fp_text reference REF** (at 0 -3.2) (layer F.SilkS)
+    (fp_text reference REF** (at 0 -3.2) (layer F.SilkS) hide
       (effects (font (size 1 1) (thickness 0.15)))
     )
@@
     (tags "mounting hole 2.2mm no annular m2")
     (attr virtual)
-    (fp_text reference REF** (at 0 -3.2) (layer F.SilkS)
-      (effects (font (size 1 1) (thickness 0.15)))
-    )
+    (fp_text reference REF** (at 0 -3.2) (layer F.SilkS) hide
+      (effects (font (size 1 1) (thickness 0.15)))
+    )
